File: PCB/airgradient-go-main/airgradient-go-main.kicad_sch (KiCad schematic)
At the start: 200 parts, among them CN1 HCZZ0032-5, CN2 HCZZ0032-5, CN3 HCZZ0032-5, Q1 SIA445EDJ-T1-GE3, Q2 ZVN4106FTA_C508255, Q3 CSD83325L, Q4 SS8050-G, Q5 SI1308EDL, SW1 TS-1091C-A1B3-D2, SW2 TS-1091C-A1B3-D2, U1 W25N512GVEIG, U10 SGP41-D-R4, U11 PS1-CO-SMOKE-10k, U12 SHT4x, U13 SPL07-003, U14 LIS2DH12TR, U15 TMUX121NKGR_C22428404, U16 S12, U17 TCA6408ARGT, U18 TAU1113, U19 LM66200DRLR, U2 ZDSD512MLGEAG, U20 LP5036, U3 BQ27742YZFR-G1, U4 ESP32-C5-MINI-1, U5 BQ25628RYKR, U6 HYG-8503A, U7 TPL5010DDCR, U8 TPS63802DLAR, U9 TPS7A0228DQNR

Commit message: No-display variant: DNP the e-paper display circuit
Same bare PCB as v2.1; only population changes. DNP parts (the whole
DISPLAY section of the schematic):
- FPC1 (display connector)
- Gate/boost circuit: Q5, L3, D3, D4, D5, C48, C54, C55, R42, R43
- Display caps: C41, C43, C45, C49, C51, C53, C58
- ePaper CS / D/C pull-ups: R39, R40

Firmware note: ePaper BUSY input to the ESP32 is left floating;
enable an internal pull or leave the pin unused.
Parts:
- C41, C43, C45, C48, C49, C51, C53, C54, C55, C58, D3, D4, D5, FPC1, L3, Q5, R39, R40, R42, R43: now not fitted
Changed lines of the file:
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@@
 		(on_board yes)
 		(in_pos_files yes)
-		(dnp no)
+		(dnp yes)
 		(fields_autoplaced yes)
 		(property "Reference" "R42"
@@
 		(on_board yes)
 		(in_pos_files yes)
-		(dnp no)
+		(dnp yes)
 		(fields_autoplaced yes)
 		(property "Reference" "R39"
@@
 		(on_board yes)
 		(in_pos_files yes)
-		(dnp no)
+		(dnp yes)
 		(fields_autoplaced yes)
 		(property "Reference" "C45"
@@
 		(on_board yes)
 		(in_pos_files yes)
-		(dnp no)
+		(dnp yes)
 		(fields_autoplaced yes)
 		(property "Reference" "D5"
@@
 		(on_board yes)
 		(in_pos_files yes)
-		(dnp no)
+		(dnp yes)
 		(fields_autoplaced yes)
 		(property "Reference" "C49"
@@
 		(on_board yes)
 		(in_pos_files yes)
-		(dnp no)
+		(dnp yes)
 		(fields_autoplaced yes)
 		(property "Reference" "L3"
@@
 		(on_board yes)
 		(in_pos_files yes)
-		(dnp no)
+		(dnp yes)
 		(fields_autoplaced yes)
 		(property "Reference" "D3"
@@
 		(on_board yes)
 		(in_pos_files yes)
-		(dnp no)
+		(dnp yes)
 		(fields_autoplaced yes)
 		(property "Reference" "C58"
@@
 		(on_board yes)
 		(in_pos_files yes)
-		(dnp no)
+		(dnp yes)
 		(fields_autoplaced yes)
 		(property "Reference" "R40"
@@
 		(on_board yes)
 		(in_pos_files yes)
-		(dnp no)
+		(dnp yes)
 		(fields_autoplaced yes)
 		(property "Reference" "C55"
@@
 		(on_board yes)
 		(in_pos_files yes)
-		(dnp no)
+		(dnp yes)
 		(fields_autoplaced yes)
 		(property "Reference" "C51"
@@
 		(on_board yes)
 		(in_pos_files yes)
-		(dnp no)
+		(dnp yes)
 		(fields_autoplaced yes)
 		(property "Reference" "C48"
@@
 		(on_board yes)
 		(in_pos_files yes)
-		(dnp no)
+		(dnp yes)
 		(fields_autoplaced yes)
 		(property "Reference" "FPC1"
@@
 		(on_board yes)
 		(in_pos_files yes)
-		(dnp no)
+		(dnp yes)
 		(fields_autoplaced yes)
 		(property "Reference" "C54"
@@
 		(on_board yes)
 		(in_pos_files yes)
-		(dnp no)
+		(dnp yes)
 		(fields_autoplaced yes)
 		(property "Reference" "R43"
@@
 		(on_board yes)
 		(in_pos_files yes)
-		(dnp no)
+		(dnp yes)
 		(fields_autoplaced yes)
 		(property "Reference" "D4"
@@
 		(on_board yes)
 		(in_pos_files yes)
-		(dnp no)
+		(dnp yes)
 		(fields_autoplaced yes)
 		(property "Reference" "C43"
@@
 		(on_board yes)
 		(in_pos_files yes)
-		(dnp no)
+		(dnp yes)
 		(fields_autoplaced yes)
 		(property "Reference" "C41"
@@
 		(on_board yes)
 		(in_pos_files yes)
-		(dnp no)
+		(dnp yes)
 		(fields_autoplaced yes)
 		(property "Reference" "Q5"
@@
 		(on_board yes)
 		(in_pos_files yes)
-		(dnp no)
+		(dnp yes)
 		(fields_autoplaced yes)
 		(property "Reference" "C53"
